File: brain-duinoV0.3/yBrainA1-11March2015.sch (EAGLE design)
At the start: 137 parts, among them IC1 OP2177ARMZ, IC2 OPA2111KP, IC3 OP4177ARZ, IC4 OPA2111KP, IC5 TLC555CDR, IC6 TAR5SB50, IC7 LT1761ES5-5, K1 AQY221R2VY, K2 AQY221R2VY

Commit message: added values to devices where ERC requires it.
Signed-off-by: Christoph Maier <cm.hardware.software.elsewhere@gmail.com>
Parts:
- AD, GND, ICSP, IOH, IOL, JP5, POWER, RXD, SJ1, SJ10, SJ11, SJ12, SJ13, SJ14, SJ15, SJ16, SJ17, SJ2, SJ3, SJ4, SJ5, SJ6, SJ7, SJ8, SJ9, TXD, VCC: value (none) -> .
Changed lines of the file:
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@@
 <?xml version="1.0" encoding="utf-8"?>
 <!DOCTYPE eagle SYSTEM "eagle.dtd">
-<eagle version="7.2.0">
+<eagle version="6.5.0">
 <drawing>
 <settings>
@@
 </classes>
 <parts>
-<part name="ICSP" library="jumper" deviceset="JP3Q" device=""/>
+<part name="ICSP" library="jumper" deviceset="JP3Q" device="" value="."/>
 <part name="C15" library="rcl" deviceset="C-EU" device="C0805" value="1µF"/>
 <part name="C11" library="rcl" deviceset="C-EU" device="C0805" value="1µF"/>
@@
 <part name="C36" library="rcl" deviceset="C-EU" device="C0805" value="47pF"/>
 <part name="GND16" library="supply1" deviceset="GND" device=""/>
-<part name="VCC" library="pinhead" deviceset="PINHD-1X1" device=""/>
-<part name="GND" library="pinhead" deviceset="PINHD-1X1" device=""/>
-<part name="TXD" library="pinhead" deviceset="PINHD-1X1" device=""/>
-<part name="RXD" library="pinhead" deviceset="PINHD-1X1" device=""/>
+<part name="VCC" library="pinhead" deviceset="PINHD-1X1" device="" value="."/>
+<part name="GND" library="pinhead" deviceset="PINHD-1X1" device="" value="."/>
+<part name="TXD" library="pinhead" deviceset="PINHD-1X1" device="" value="."/>
+<part name="RXD" library="pinhead" deviceset="PINHD-1X1" device="" value="."/>
 <part name="GND8" library="supply1" deviceset="GND" device=""/>
 <part name="IC3" library="linear" deviceset="TL064" device="D" value="OP4177ARZ"/>
-<part name="IOH" library="pinhead" deviceset="PINHD-1X10" device=""/>
-<part name="POWER" library="pinhead" deviceset="PINHD-1X8" device=""/>
-<part name="AD" library="pinhead" deviceset="PINHD-1X6" device=""/>
-<part name="IOL" library="pinhead" deviceset="PINHD-1X8" device=""/>
+<part name="IOH" library="pinhead" deviceset="PINHD-1X10" device="" value="."/>
+<part name="POWER" library="pinhead" deviceset="PINHD-1X8" device="" value="."/>
+<part name="AD" library="pinhead" deviceset="PINHD-1X6" device="" value="."/>
+<part name="IOL" library="pinhead" deviceset="PINHD-1X8" device="" value="."/>
 <part name="R20" library="rcl" deviceset="R-EU_" device="R0805" value="470"/>
 <part name="R22" library="rcl" deviceset="R-EU_" device="R0805" value="1K"/>
@@
 <part name="C39" library="rcl" deviceset="C-EU" device="C0805" value="10µF"/>
 <part name="S2" library="switch-misc" deviceset="9450-2" device=""/>
-<part name="SJ1" library="jumper" deviceset="SJ2W" device=""/>
-<part name="SJ2" library="jumper" deviceset="SJ2W" device=""/>
-<part name="SJ3" library="jumper" deviceset="SJ2W" device=""/>
+<part name="SJ1" library="jumper" deviceset="SJ2W" device="" value="."/>
+<part name="SJ2" library="jumper" deviceset="SJ2W" device="" value="."/>
+<part name="SJ3" library="jumper" deviceset="SJ2W" device="" value="."/>
 <part name="C40" library="rcl" deviceset="C-EU" device="C0805" value="0.1µF"/>
 <part name="C41" library="rcl" deviceset="C-EU" device="C0805" value="0.1µF"/>
@@
 <part name="R29" library="rcl" deviceset="R-EU_" device="R0805" value="2.15K"/>
 <part name="K1" library="relay" deviceset="AQY221*2V" device="" technology="R" value="AQY221R2VY"/>
-<part name="SJ4" library="jumper" deviceset="SJ2W" device=""/>
-<part name="SJ5" library="jumper" deviceset="SJ2W" device=""/>
+<part name="SJ4" library="jumper" deviceset="SJ2W" device="" value="."/>
+<part name="SJ5" library="jumper" deviceset="SJ2W" device="" value="."/>
 <part name="C44" library="rcl" deviceset="C-EU" device="C0805" value="15nF"/>
 <part name="C45" library="rcl" deviceset="C-EU" device="C0805" value="2.7nF"/>
@@
 <part name="C47" library="rcl" deviceset="C-EU" device="C0805" value="1µF"/>
 <part name="D2" library="diode" deviceset="PD3S160" device="" value="RB160M-30"/>
-<part name="SJ7" library="jumper" deviceset="SJ2W" device=""/>
+<part name="SJ7" library="jumper" deviceset="SJ2W" device="" value="."/>
 <part name="GND19" library="supply1" deviceset="GND" device=""/>
-<part name="SJ8" library="jumper" deviceset="SJ2W" device=""/>
+<part name="SJ8" library="jumper" deviceset="SJ2W" device="" value="."/>
 <part name="C48" library="rcl" deviceset="C-EU" device="C0805" value="0.1µF"/>
 <part name="C49" library="rcl" deviceset="C-EU" device="C0805" value="0.1µF"/>
 <part name="GND25" library="supply1" deviceset="GND" device=""/>
 <part name="GND26" library="supply1" deviceset="GND" device=""/>
-<part name="SJ9" library="jumper" deviceset="SJ2W" device=""/>
+<part name="SJ9" library="jumper" deviceset="SJ2W" device="" value="."/>
 <part name="C50" library="rcl" deviceset="C-EU" device="C0805" value="0.1µF"/>
 <part name="C51" library="rcl" deviceset="C-EU" device="C0805" value="0.1µF"/>
 <part name="GND27" library="supply1" deviceset="GND" device=""/>
-<part name="SJ10" library="jumper" deviceset="SJ" device=""/>
-<part name="SJ11" library="jumper" deviceset="SJ" device=""/>
+<part name="SJ10" library="jumper" deviceset="SJ" device="" value="."/>
+<part name="SJ11" library="jumper" deviceset="SJ" device="" value="."/>
 <part name="U$1" library="MKH" deviceset="AD8220" device="" value="AD8422ARMZ"/>
 <part name="U$2" library="MKH" deviceset="AD8220" device="" value="AD8422ARMZ"/>
 <part name="IC1" library="analog-devices" deviceset="AD8656" device="RM" value="OP2177ARMZ"/>
-<part name="SJ12" library="jumper" deviceset="SJ" device=""/>
-<part name="SJ13" library="jumper" deviceset="SJ" device=""/>
-<part name="SJ14" library="jumper" deviceset="SJ" device=""/>
-<part name="SJ15" library="jumper" deviceset="SJ" device=""/>
-<part name="SJ16" library="jumper" deviceset="SJ" device=""/>
-<part name="SJ6" library="jumper" deviceset="SJ" device=""/>
-<part name="SJ17" library="jumper" deviceset="SJ" device=""/>
-<part name="JP5" library="pinhead" deviceset="PINHD-2X5" device="/90"/>
+<part name="SJ12" library="jumper" deviceset="SJ" device="" value="."/>
+<part name="SJ13" library="jumper" deviceset="SJ" device="" value="."/>
+<part name="SJ14" library="jumper" deviceset="SJ" device="" value="."/>
+<part name="SJ15" library="jumper" deviceset="SJ" device="" value="."/>
+<part name="SJ16" library="jumper" deviceset="SJ" device="" value="."/>
+<part name="SJ6" library="jumper" deviceset="SJ" device="" value="."/>
+<part name="SJ17" library="jumper" deviceset="SJ" device="" value="."/>
+<part name="JP5" library="pinhead" deviceset="PINHD-2X5" device="/90" value="."/>
 </parts>
 <sheets>
@@
 <wire x1="68.58" y1="53.34" x2="68.58" y2="45.72" width="0.1524" layer="91"/>
 <wire x1="10.16" y1="45.72" x2="15.24" y2="45.72" width="0.1524" layer="91"/>
-<wire x1="15.24" y1="45.72" x2="68.58" y2="45.72" width="0.1524" layer="91"/>
+<wire x1="15.24" y1="45.72" x2="55.88" y2="45.72" width="0.1524" layer="91"/>
+<wire x1="55.88" y1="45.72" x2="68.58" y2="45.72" width="0.1524" layer="91"/>
 <wire x1="68.58" y1="45.72" x2="68.58" y2="40.64" width="0.1524" layer="91"/>
 <pinref part="C18" gate="G$1" pin="1"/>
@@
 <wire x1="15.24" y1="60.96" x2="15.24" y2="45.72" width="0.1524" layer="91"/>
 <junction x="15.24" y="45.72"/>
+<pinref part="JP5" gate="A" pin="5"/>
+<wire x1="43.18" y1="60.96" x2="15.24" y2="60.96" width="0.1524" layer="91"/>
 <pinref part="JP5" gate="A" pin="6"/>
-<pinref part="JP5" gate="A" pin="5"/>
-<wire x1="50.8" y1="60.96" x2="43.18" y2="60.96" width="0.1524" layer="91"/>
-<wire x1="43.18" y1="60.96" x2="15.24" y2="60.96" width="0.1524" layer="91"/>
+<wire x1="50.8" y1="60.96" x2="55.88" y2="60.96" width="0.1524" layer="91"/>
+<wire x1="55.88" y1="60.96" x2="55.88" y2="45.72" width="0.1524" layer="91"/>
+<junction x="55.88" y="45.72"/>
 </segment>
 <segment>
